File: hexpansion.kicad_pcb (KiCad board)
At the start: 2 copper layers, 32 x 36.6 mm, 4 parts, among them J1 Hexpansion-Connector, U2 XIAO-ESP32-S3-DIP

Commit message: Add files via upload
Parts:
- added R1: R, Resistor_SMD:R_0805_2012Metric, F.Cu at (112.6, 101.1)
- added R2: R, Resistor_SMD:R_0805_2012Metric, F.Cu at (109.3, 101.1)
- added U1: XIAO-ESP32-S3-DIP, XIAO:XIAO-ESP32-S3-DIP, F.Cu at (127.0, 99.7)
- U2: value XIAO-ESP32-S3-DIP -> FM24CL16B; footprint XIAO:XIAO-ESP32-S3-DIP -> Package_SO:SOIC-8_3.9x4.9mm_P1.27mm
- moved U2 17.5 mm to (111.1, 107.1), turned to 180 degrees
Connections:
- U2 pad 4: unconnected-(U2-PA11_A3_D3-Pad4) -> /GND
- U2 pad 5: unconnected-(U2-PA8_A4_D4_SDA-Pad5) -> /SDA
- U2 pad 6: unconnected-(U2-PA9_A5_D5_SCL-Pad6) -> /SCL
- U2 pad 8: unconnected-(U2-PB09_A7_D7_RX-Pad8) -> /3V3
Routing:
- net /GND: track 232.1 -> 58.6 mm, vias 2 -> 7
- net /3V3: track 103.5 -> 49.6 mm, vias 1 -> 0
- net /LS_E: track 27.2 -> 0.00 mm
- net /LS_D: track 26.1 -> 0.00 mm
- net unconnected-(J1-LS_A-Pad2): track 25.9 -> 0.00 mm
- net /LS_C: track 25.5 -> 0.00 mm
- net unconnected-(J1-LS_B-Pad3): track 25.2 -> 0.00 mm
- net /HS_G: track 22.7 -> 0.00 mm
- net /HS_H: track 22.5 -> 0.00 mm
- net (no net): track 9.71 -> 0.00 mm
- net /SCL: track 24.0 -> 15.2 mm, vias 0 -> 1
- net /SDA: track 24.5 -> 16.0 mm, vias 0 -> 1
- net /HS_I: track 23.2 -> 24.6 mm
- net /HS_F: track 23.4 -> 22.8 mm
Other:
- board size 32 x 36.6 mm -> 37.7 x 36.6 mm
