File: hexpansion.kicad_sch (KiCad schematic)
At the start: 4 parts, among them J1 Hexpansion-Connector, U1 XIAO-ESP32-S3-DIP

Commit message: Add files via upload
Parts:
- added R1, R2: R, Resistor_SMD:R_0805_2012Metric, symbol Device:R
- added U2: FM24CL16B, Package_SO:SOIC-8_3.9x4.9mm_P1.27mm, symbol Memory_NVRAM:FM24CL16B
Connections:
- net 3V3: now also R1.1, R2.1, U2.8 (VDD)
- net GND: now also U2.4 (VSS)
- net HS_H: now also U1.7 (PB08_A6_D6_TX)
- net HS_I: now also U1.8 (PB09_A7_D7_RX)
- net SCL: now also R2.2, U2.6 (SCL)
- net SDA: now also R1.2, U2.5 (SDA)
- no-connect marks 0 -> 9
